File: kicad/map2.sch (KiCad schematic (older format))
At the start: 18 parts, among them P1 5V, P2 5V, P4 GND, P5 GND, P7 MTG, P8 MTG, P9 LOGO, Q1 2N2222

Commit message: work in progress
Parts:
- BT1: manf# (none) -> mfr_pn
- P9: footprint (none) -> map2:MA_logo
- Q1: footprint map2:TO-92-Bipolar-rugged-CBE -> map2:TO-92_Molded_Narrow
Connections:
- net 5V: now reaches BT1.+, D1.1 (A), P1.1 (P1), P2.1 (P1), R1.1, R2.1, R3.1
- net LDR: now reaches C1.2 (-), R1.2, R5.1
- net BASE: now reaches C1.1 (+), C2.2 (-), Q1.2 (B), R2.2
- net at C2.1 (+), R3.2: now also C3.1 (+); no longer C3.2 (-)
- net LED: now reaches D1.2 (K), R4.1
- net COLL: now reaches Q1.1 (C), R4.2
- net COLL: now also C3.2 (-); no longer C3.1 (+)
- net GND: now reaches BT1.-, P4.1 (P1), P5.1 (P1), Q1.3 (E), R5.2
Other:
- moved on the sheet: C3
Changed lines of the file:
@@
 EESchema Schematic File Version 2
-LIBS:mmM
+LIBS:map2
 LIBS:power
 LIBS:map2-cache
@@
 L C_POL_1 C3
 U 1 1 56D18ACF
-P 4025 2575
-F 0 "C3" V 3975 2600 40  0000 L CNB
-F 1 "47uF" V 4150 2575 40  0000 L CNN
-F 2 "map2:Capacitor5x6RM2.5" H 4025 2575 60  0001 C CNN
-F 3 "" H 4025 2575 60  0000 C CNN
-F 4 "CAP ALUM 100UF 16V 20% RADIAL" H 4025 2775 60  0001 L CNN "Field4"
-F 5 "100u,16V" H 4025 2875 60  0001 L CNN "Field5"
-F 6 "Radial, Can, 6.3mm dia" H 4025 2975 60  0001 L CNN "Field6"
-F 7 "Panasonic Electronic Components" H 4025 3075 60  0001 L CNN "Field7"
-F 8 "ECE-A1CKA101" H 4025 3175 60  0001 L CNN "Field8"
-F 9 "Digikey" H 4025 3275 60  0001 L CNN "Field9"
-F 10 "P833-ND" H 4025 3375 60  0001 L CNN "Field10"
-F 11 "http://www.digikey.com/product-detail/en/ECE-A1CKA101/P833-ND/44757?cur=USD" H 4025 3475 60  0001 L CNN "Field11"
-	1    4025 2575
-	0    1    1    0
+P 3975 2575
+F 0 "C3" V 3925 2600 40  0000 L CNB
+F 1 "47uF" V 4100 2575 40  0000 L CNN
+F 2 "map2:Capacitor5x6RM2.5" H 3975 2575 60  0001 C CNN
+F 3 "" H 3975 2575 60  0000 C CNN
+F 4 "CAP ALUM 100UF 16V 20% RADIAL" H 3975 2775 60  0001 L CNN "Field4"
+F 5 "100u,16V" H 3975 2875 60  0001 L CNN "Field5"
+F 6 "Radial, Can, 6.3mm dia" H 3975 2975 60  0001 L CNN "Field6"
+F 7 "Panasonic Electronic Components" H 3975 3075 60  0001 L CNN "Field7"
+F 8 "ECE-A1CKA101" H 3975 3175 60  0001 L CNN "Field8"
+F 9 "Digikey" H 3975 3275 60  0001 L CNN "Field9"
+F 10 "P833-ND" H 3975 3375 60  0001 L CNN "Field10"
+F 11 "http://www.digikey.com/product-detail/en/ECE-A1CKA101/P833-ND/44757?cur=USD" H 3975 3475 60  0001 L CNN "Field11"
+	1    3975 2575
+	0    -1   -1   0
 $EndComp
 $Comp
@@
 F 0 "Q1" H 4350 3175 40  0000 L CNB
 F 1 "2N2222" H 4350 3100 40  0000 L CNN
-F 2 "map2:TO-92-Bipolar-rugged-CBE" H 4340 3175 30  0001 C CNN
+F 2 "map2:TO-92_Molded_Narrow" H 4340 3175 30  0001 C CNN
 F 3 "" H 4150 3175 60  0000 C CNN
 	1    4150 3175
@@
 F 0 "P9" V 1650 5175 50  0000 C CNB
 F 1 "LOGO" V 1850 5100 50  0000 C CNN
-F 2 "" H 1750 5100 50  0001 C CNN
+F 2 "map2:MA_logo" H 1750 5100 50  0001 C CNN
 F 3 "" H 1750 5100 50  0000 C CNN
 	1    1750 5100
@@
 F 2 "" H 1750 2625 60  0001 C CNN
 F 3 "" H 1750 2625 60  0000 C CNN
-F 4 "HOLDER BATTERY COIN 20MM DIA THM" H 1750 2925 60  0001 L CNN "Field4"
-F 5 "Coin Cell, Retainer" H 1750 3025 60  0001 L CNN "Field5"
-F 6 "Coin, 20.0mm" H 1750 3125 60  0001 L CNN "Field6"
-F 7 "Keystone Electronics" H 1750 3225 60  0001 L CNN "Field7"
-F 8 "3003" H 1750 3325 60  0001 L CNN "Field8"
-F 9 "Digikey" H 1750 3425 60  0001 L CNN "Field9"
-F 10 "3003K-ND" H 1750 3525 60  0001 L CNN "Field10"
-F 11 "http://www.digikey.com/scripts/DkSearch/dksus.dll?x=0&y=0&lang=en&KeyWords=3003K-ND&cur=USD" H 1750 3625 60  0001 L CNN "Field11"
+F 4 "mfr_pn" H 1750 2625 60  0001 C CNN "manf#"
+F 5 "HOLDER BATTERY COIN 20MM DIA THM" H 1750 2925 60  0001 L CNN "Field4"
+F 6 "Coin Cell, Retainer" H 1750 3025 60  0001 L CNN "Field5"
+F 7 "Coin, 20.0mm" H 1750 3125 60  0001 L CNN "Field6"
+F 8 "Keystone Electronics" H 1750 3225 60  0001 L CNN "Field7"
+F 9 "3003" H 1750 3325 60  0001 L CNN "Field8"
+F 10 "Digikey" H 1750 3425 60  0001 L CNN "Field9"
+F 11 "3003K-ND" H 1750 3525 60  0001 L CNN "Field10"
+F 12 "http://www.digikey.com/scripts/DkSearch/dksus.dll?x=0&y=0&lang=en&KeyWords=3003K-ND&cur=USD" H 1750 3625 60  0001 L CNN "Field11"
 	1    1750 2625
 	0    1    1    0
@@
 	1    0    0    -1
 $EndComp
+Text Label 2750 2825 0    40   ~ 0
+LDR
+Text Label 3375 3175 0    40   ~ 0
+BASE
+Text Label 4250 2775 0    40   ~ 0
+COLL
+Text Label 4250 1925 0    40   ~ 0
+LED
+Text Label 2225 1250 0    40   ~ 0
+5V
+Text Label 2275 3725 0    40   ~ 0
+GND
 $EndSCHEMATC

Commit message: gerbers ready
Parts:
- P7, P8: footprint map2:MountingHole_3mm -> map2:MTG_3mm
- R5: value R_photo -> LDR
Connections:
- net 5V: now also P8.1 (P1)
- net GND: now also P7.1 (P1)
- no-connect marks 3 -> 1
Other:
- moved on the sheet: P7, P8
Changed lines of the file:
@@
 EELAYER 25 0
 EELAYER END
-$Descr A4 11693 8268
+$Descr User 8270 5840
 encoding utf-8
 Sheet 1 1
@@
 $EndDescr
 $Bitmap
-Pos 10425 6850
+Pos 7000 4400
 Scale 0.200000
 Data
@@
 L CONN_01X01 P7
 U 1 1 56D1A7FC
-P 1250 5100
-F 0 "P7" V 1150 5175 50  0000 C CNB
-F 1 "MTG" V 1350 5100 50  0000 C CNN
-F 2 "map2:MountingHole_3mm" H 1250 5100 50  0001 C CNN
-F 3 "" H 1250 5100 50  0000 C CNN
-	1    1250 5100
-	0    1    1    0
+P 1250 3375
+F 0 "P7" V 1150 3450 50  0000 C CNB
+F 1 "MTG" V 1350 3375 50  0000 C CNN
+F 2 "map2:MTG_3mm" H 1250 3375 50  0001 C CNN
+F 3 "" H 1250 3375 50  0000 C CNN
+	1    1250 3375
+	0    -1   -1   0
 $EndComp
 $Comp
 L CONN_01X01 P8
 U 1 1 56D1A8D9
-P 1500 5100
-F 0 "P8" V 1400 5175 50  0000 C CNB
-F 1 "MTG" V 1600 5100 50  0000 C CNN
-F 2 "map2:MountingHole_3mm" H 1500 5100 50  0001 C CNN
-F 3 "" H 1500 5100 50  0000 C CNN
-	1    1500 5100
+P 1250 1600
+F 0 "P8" V 1150 1675 50  0000 C CNB
+F 1 "MTG" V 1350 1600 50  0000 C CNN
+F 2 "map2:MTG_3mm" H 1250 1600 50  0001 C CNN
+F 3 "" H 1250 1600 50  0000 C CNN
+	1    1250 1600
 	0    1    1    0
 $EndComp
-NoConn ~ 1250 4900
-NoConn ~ 1500 4900
 $Comp
 L CONN_01X01 P9
@@
 $EndComp
 Wire Wire Line
-	1250 1125 1250 1250
+	1250 1125 1250 1400
 Connection ~ 1750 1250
 $Comp
@@
 $EndComp
 Wire Wire Line
-	1250 3725 1250 3850
+	1250 3575 1250 3850
 Connection ~ 1750 3725
 $Comp
@@
 P 2750 3175
 F 0 "R5" H 2800 3325 40  0000 C CNB
-F 1 "R_photo" V 2925 3175 40  0000 C CNN
+F 1 "LDR" H 2825 3000 40  0000 C CNN
 F 2 "map2:R_photo" H 2750 3175 60  0001 C CNN
 F 3 "" H 2750 3175 60  0000 C CNN
@@
 Text Label 2275 3725 0    40   ~ 0
 GND
+Connection ~ 1250 3725
+Connection ~ 1250 1250
 $EndSCHEMATC
