File: kicad/map2_smd.kicad_pcb (KiCad board)
At the start: 2 copper layers, 25.4 x 25.4 mm, 31 parts, among them P1 5V, P2 5V, P4 GND, P5 GND, P7 MTG, P8 MTG, P9 LOGO, Q1 2N2222

Commit message: _smd version gerbers
Parts:
- moved Q1 1.14 mm to (37.3, 35.8), turned to 180 degrees
Connections:
- Q1 pad 1: /BASE -> /COLL
- Q1 pad 2: /COLL -> /BASE
Routing:
- net /COLL: track 25.8 -> 33.2 mm
- net /BASE: track 52.2 -> 46.8 mm
- net Net-(C2-Pad1): track 35.9 -> 35.0 mm
- net /GND: track 70.4 -> 69.8 mm
