File: kicad/map2_smd.kicad_pcb (KiCad board)
At the start: 2 copper layers, 25.4 x 25.4 mm, 31 parts, among them P1 5V, P2 5V, P4 GND, P5 GND, P7 MTG, P8 MTG, P9 LOGO, Q1 2N2222

Commit message: working on 3D cad layout
Parts:
- removed P2: 5V, map2:Pin_Header_Straight_1x01
- removed P5: GND, map2:Pin_Header_Straight_1x01
- P1, P4: footprint map2:Pin_Header_Straight_1x01 -> map2:Pin_Header_Straight_1x02
- P9: footprint map2:MA_logo -> map2:MA_LOGO
- moved P1 1.27 mm to (36.8, 42.5), turned to 180 degrees
- moved P4 1.27 mm to (54.6, 42.5), turned to 180 degrees

Commit message: update
Parts:
- removed the via1 at (58.4, 52.7)
- removed the via1 at (58.4, 50.2)
- removed the via1 at (58.4, 47.6)
- removed the via2 at (33.0, 52.7)
- removed the via2 at (33.0, 50.2)
- removed the via2 at (33.0, 47.6)
Routing:
- net /5V: track 61.2 -> 52.0 mm
- net /GND: track 69.8 -> 75.1 mm
