File: kicad/map2_smd.sch (KiCad schematic (older format))
At the start: 18 parts, among them P1 5V, P2 5V, P4 GND, P5 GND, P7 MTG, P8 MTG, P9 LOGO, Q1 2N2222

Commit message: working on 3D cad layout
Parts:
- removed P1: 5V, map2:Pin_Header_Straight_1x01, symbol CONN_01X01
- removed P4: GND, map2:Pin_Header_Straight_1x01, symbol CONN_01X01
- added P1: 5V, map2:Pin_Header_Straight_1x02, symbol CONN_01X02
- added P4: GND, map2:Pin_Header_Straight_1x02, symbol CONN_01X02
- P2, P5: footprint map2:Pin_Header_Straight_1x01 -> (none); manf# (none) -> mfr_pn
- P9: footprint (none) -> map2:MA_LOGO
Connections:
- net 5V: now also P1.1 (P1), P1.2 (P2)
- net GND: now also P4.1 (P1), P4.2 (P2)
Changed lines of the file:
@@
 LIBS:map2
 LIBS:power
+LIBS:conn
 LIBS:map2_smd-cache
 EELAYER 25 0
@@
 	2750 1250 2750 1950
 Wire Wire Line
-	1250 1250 4250 1250
+	1150 1250 4250 1250
 Wire Wire Line
 	4250 1250 4250 1400
@@
 	4250 3725 4250 3375
 Wire Wire Line
-	1250 3725 4250 3725
+	1150 3725 4250 3725
 Wire Wire Line
 	2750 3725 2750 3425
@@
 F 0 "P2" V 1650 875 50  0000 C CNB
 F 1 "5V" V 1850 925 50  0000 C CNN
-F 2 "map2:Pin_Header_Straight_1x01" H 1750 925 50  0001 C CNN
+F 2 "" H 1750 925 50  0001 C CNN
 F 3 "" H 1750 925 50  0000 C CNN
+F 4 "mfr_pn" H 1750 925 60  0001 C CNN "manf#"
 	1    1750 925
 	0    -1   -1   0
@@
 F 0 "P5" V 1650 4125 50  0000 C CNB
 F 1 "GND" V 1850 4050 50  0000 C CNN
-F 2 "map2:Pin_Header_Straight_1x01" H 1750 4050 50  0001 C CNN
+F 2 "" H 1750 4050 50  0001 C CNN
 F 3 "" H 1750 4050 50  0000 C CNN
+F 4 "mfr_pn" H 1750 4050 60  0001 C CNN "manf#"
 	1    1750 4050
 	0    1    1    0
@@
 	0    1    1    0
 $EndComp
-$Comp
-L CONN_01X01 P1
-U 1 1 56D1AA9B
-P 1250 925
-F 0 "P1" V 1150 875 50  0000 C CNB
-F 1 "5V" V 1350 925 50  0000 C CNN
-F 2 "map2:Pin_Header_Straight_1x01" H 1250 925 50  0001 C CNN
-F 3 "" H 1250 925 50  0000 C CNN
-	1    1250 925
-	0    -1   -1   0
-$EndComp
 Wire Wire Line
 	1250 1125 1250 1400
 Connection ~ 1750 1250
-$Comp
-L CONN_01X01 P4
-U 1 1 56D1AC34
-P 1250 4050
-F 0 "P4" V 1150 4125 50  0000 C CNB
-F 1 "GND" V 1350 4050 50  0000 C CNN
-F 2 "map2:Pin_Header_Straight_1x01" H 1250 4050 50  0001 C CNN
-F 3 "" H 1250 4050 50  0000 C CNN
-	1    1250 4050
-	0    1    1    0
-$EndComp
 Wire Wire Line
 	1250 3575 1250 3850
@@
 F 0 "P9" V 1425 5100 50  0000 C CNB
 F 1 "LOGO" V 1625 5100 50  0000 C CNN
-F 2 "" H 1525 5100 50  0000 C CNN
+F 2 "map2:MA_LOGO" H 1525 5100 50  0001 C CNN
 F 3 "" H 1525 5100 50  0000 C CNN
 	1    1525 5100
 	0    1    1    0
 $EndComp
+$Comp
+L CONN_01X02 P4
+U 1 1 56D85B2F
+P 1200 4050
+F 0 "P4" V 1100 4175 50  0000 C CNB
+F 1 "GND" V 1300 4050 50  0000 C CNN
+F 2 "map2:Pin_Header_Straight_1x02" H 1200 4050 50  0001 C CNN
+F 3 "" H 1200 4050 50  0000 C CNN
+	1    1200 4050
+	0    1    1    0
+$EndComp
+Wire Wire Line
+	1150 3850 1150 3725
+$Comp
+L CONN_01X02 P1
+U 1 1 56D85E47
+P 1200 925
+F 0 "P1" V 1100 825 50  0000 C CNB
+F 1 "5V" V 1300 925 50  0000 C CNN
+F 2 "map2:Pin_Header_Straight_1x02" H 1200 925 50  0001 C CNN
+F 3 "" H 1200 925 50  0000 C CNN
+	1    1200 925
+	0    -1   -1   0
+$EndComp
+Wire Wire Line
+	1150 1125 1150 1250
 $EndSCHEMATC
